File: SAE-Cellular-Module/SAE Cellular Module.kicad_sch (KiCad schematic)
At the start: 1 part, among them J1 Microfit 3.0

Commit message: Added initial component placements
Parts:
- J1: footprint (none) -> 436500428:CONN_SD-43650-010_04_MOL; MPN (none) -> 0436500428
